File: kicad_files/toasty-tkl.sch (KiCad schematic (older format))
At the start: 195 parts, among them CON1 USB-MINI-B, SW0:0 ESC, SW0:10 F9, SW0:11 F10, SW0:12 F11, SW0:13 F12, SW0:14 PRINT, SW0:15 SCROLL LOCK, SW0:2 F1, SW0:3 F2, SW0:4 F3, SW0:5 F4, SW0:6 F5, SW0:7 F6, SW0:8 F7, SW0:9 F8, SW1:0 `, SW1:1 1, SW1:10 0, SW1:11 -, SW1:12 =, SW1:13 BACK SPACE, SW1:14 INSERT, SW1:15 HOME, SW1:2 2, SW1:3 3, SW1:4 4, SW1:5 5, SW1:6 6, SW1:7 7, SW1:8 8, SW1:9 9, SW2:0 TAB, SW2:1 Q, SW2:10 P, SW2:11 [, SW2:12 ], SW2:13 \\, SW2:14 DELETE, SW2:15 END, SW2:2 W, SW2:3 E, SW2:4 R, SW2:5 T, SW2:6 Y, SW2:7 U, SW2:8 I, SW2:9 O, SW3:0 CAPS LOCK, SW3:1 A, SW3:10 ;, SW3:11 ', SW3:13 ENTER, SW3:14 PAGE UP, SW3:15 PAUSE, SW3:2 S, SW3:3 D, SW3:4 F, SW3:5 G, SW3:6 H, SW3:7 J, SW3:8 K, SW3:9 L, SW4:0 LEFT SHIFT, SW4:1 Z, SW4:10 /, SW4:13 RIGHT SHIFT, SW4:14 PAGE DOWN, SW4:15 UP, SW4:2 X, SW4:3 C, SW4:4 V, SW4:5 B, SW4:6 N, SW4:7 M, SW4:8 ,, SW4:9 ., SW5:0 LEFT CTRL, SW5:1 LEFT WINDOWS, SW5:10 RIGHT WINDOWS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

Commit message: Added more information on LED notes including parts.
Parts:
- removed FET1: ZVN4206AV, symbol FQPF13N06L
- added C? (x3): CP1, ~, symbol CP1
- added D?: DIODE, ~, symbol DIODE
- added L?: INDUCTOR, ~, symbol INDUCTOR
- added Q?: FET_N, ~, symbol FET_N
- added R? (x4): RESISTOR, ~, symbol RESISTOR
- VREG1: symbol MC34063ABN -> MC34063
Connections:
- wire segments 629 -> 633
Other:
- moved on the sheet: F1
Changed lines of the file:
@@
-EESchema Schematic File Version 2
+EESchema Schematic File Version 2  date 16/06/2013 8:00:48 PM
 LIBS:components
 LIBS:toasty-tkl-cache
@@
 Sheet 1 1
 Title "Toasty TKL"
-Date "14 jun 2013"
+Date "17 jun 2013"
 Rev "REV 1A"
 Comp ""
@@
 LEDCOL10
 $Comp
-L MC34063ABN VREG1
+L MC34063 VREG1
 U 1 1 519C1E60
-P -750 7200
-F 0 "VREG1" H -750 7550 60  0000 C CNN
-F 1 "MC34063ABN" H -750 6850 60  0000 C CNN
-F 2 "" H -750 7200 60  0000 C CNN
-F 3 "" H -750 7200 60  0000 C CNN
-	1    -750 7200
+P -1650 8800
+F 0 "VREG1" H -1650 9150 60  0000 C CNN
+F 1 "MC34063ABN" H -1650 8450 60  0000 C CNN
+F 2 "" H -1650 8800 60  0000 C CNN
+F 3 "" H -1650 8800 60  0000 C CNN
+	1    -1650 8800
 	-1   0    0    1
 $EndComp
@@
 $EndComp
 $Comp
-L FQPF13N06L FET1
-U 1 1 519C45FB
-P 9900 -2900
-F 0 "FET1" H 9900 -3200 60  0000 C CNN
-F 1 "ZVN4206AV" H 9950 -2600 60  0000 C CNN
-F 2 "" H 9900 -2900 60  0000 C CNN
-F 3 "" H 9900 -2900 60  0000 C CNN
-	1    9900 -2900
+L FUSE F1
+U 1 1 519CE3F5
+P -1650 10900
+F 0 "F1" H -1650 10750 60  0000 C CNN
+F 1 "FUSE" H -1650 11050 60  0000 C CNN
+F 2 "" H -1650 10900 60  0000 C CNN
+F 3 "" H -1650 10900 60  0000 C CNN
+	1    -1650 10900
+	0    -1   -1   0
+$EndComp
+$Comp
+L USB-MINI-B CON1
+U 1 1 51BB5678
+P 5000 -2300
+F 0 "CON1" H 4750 -1850 60  0000 C CNN
+F 1 "USB-MINI-B" H 4950 -2800 60  0000 C CNN
+F 2 "" H 5000 -2300 60  0000 C CNN
+F 3 "" H 5000 -2300 60  0000 C CNN
+	1    5000 -2300
 	1    0    0    -1
 $EndComp
+Text Label 17600 7700 2    60   ~ 0
+GND
 $Comp
-L FUSE F1
-U 1 1 519CE3F5
-P -650 8050
-F 0 "F1" H -650 7900 60  0000 C CNN
-F 1 "FUSE" H -650 8200 60  0000 C CNN
-F 2 "" H -650 8050 60  0000 C CNN
-F 3 "" H -650 8050 60  0000 C CNN
-	1    -650 8050
+L USB-MINI-B_EXT U1
+U 1 1 51BB56F7
+P 3600 -2300
+F 0 "U1" H 3600 -1850 60  0000 C CNN
+F 1 "USB-MINI-B_EXT" H 3600 -2800 60  0000 C CNN
+F 2 "" H 3600 -2300 60  0000 C CNN
+F 3 "" H 3600 -2300 60  0000 C CNN
+	1    3600 -2300
+	1    0    0    -1
+$EndComp
+$Comp
+L FET_N Q?
+U 1 1 51BE4888
+P 9850 -3300
+F 0 "Q?" H 9753 -3050 70  0000 C CNN
+F 1 "FET_N" H 9703 -3547 60  0000 C CNN
+F 2 "~" H 9850 -3300 60  0000 C CNN
+F 3 "~" H 9850 -3300 60  0000 C CNN
+	1    9850 -3300
+	0    -1   1    0
+$EndComp
+$Comp
+L CP1 C?
+U 1 1 51BE5B22
+P -1650 6700
+F 0 "C?" H -1600 6800 50  0000 L CNN
+F 1 "CP1" H -1600 6600 50  0000 L CNN
+F 2 "~" H -1650 6700 60  0000 C CNN
+F 3 "~" H -1650 6700 60  0000 C CNN
+	1    -1650 6700
+	-1   0    0    1
+$EndComp
+$Comp
+L CP1 C?
+U 1 1 51BE5B31
+P -1650 9900
+F 0 "C?" H -1600 10000 50  0000 L CNN
+F 1 "CP1" H -1600 9800 50  0000 L CNN
+F 2 "~" H -1650 9900 60  0000 C CNN
+F 3 "~" H -1650 9900 60  0000 C CNN
+	1    -1650 9900
+	1    0    0    -1
+$EndComp
+$Comp
+L CP1 C?
+U 1 1 51BE5B40
+P -150 8650
+F 0 "C?" H -100 8750 50  0000 L CNN
+F 1 "CP1" H -100 8550 50  0000 L CNN
+F 2 "~" H -150 8650 60  0000 C CNN
+F 3 "~" H -150 8650 60  0000 C CNN
+	1    -150 8650
+	0    -1   -1   0
+$EndComp
+$Comp
+L RESISTOR R?
+U 1 1 51BE5B4F
+P -3000 9000
+F 0 "R?" V -3000 8900 50  0000 C CNN
+F 1 "RESISTOR" V -3000 9100 50  0000 C CNN
+F 2 "~" H -3000 9000 60  0000 C CNN
+F 3 "~" H -3000 9000 60  0000 C CNN
+	1    -3000 9000
+	0    -1   -1   0
+$EndComp
+$Comp
+L RESISTOR R?
+U 1 1 51BE5B5E
+P 0 10000
+F 0 "R?" V 0   9900 50  0000 C CNN
+F 1 "RESISTOR" V 0   10100 50  0000 C CNN
+F 2 "~" H 0   10000 60  0000 C CNN
+F 3 "~" H 0   10000 60  0000 C CNN
+	1    0    10000
+	1    0    0    -1
+$EndComp
+$Comp
+L RESISTOR R?
+U 1 1 51BE5B6D
+P 250 10000
+F 0 "R?" V 250 9900 50  0000 C CNN
+F 1 "RESISTOR" V 250 10100 50  0000 C CNN
+F 2 "~" H 250 10000 60  0000 C CNN
+F 3 "~" H 250 10000 60  0000 C CNN
+	1    250  10000
+	1    0    0    -1
+$EndComp
+$Comp
+L RESISTOR R?
+U 1 1 51BE5B7C
+P 500 10000
+F 0 "R?" V 500 9900 50  0000 C CNN
+F 1 "RESISTOR" V 500 10100 50  0000 C CNN
+F 2 "~" H 500 10000 60  0000 C CNN
+F 3 "~" H 500 10000 60  0000 C CNN
+	1    500  10000
+	1    0    0    -1
+$EndComp
+$Comp
+L INDUCTOR L?
+U 1 1 51BE5B8B
+P -3700 8900
+F 0 "L?" V -3750 8900 40  0000 C CNN
+F 1 "INDUCTOR" V -3600 8900 40  0000 C CNN
+F 2 "~" H -3700 8900 60  0000 C CNN
+F 3 "~" H -3700 8900 60  0000 C CNN
+	1    -3700 8900
 	0    -1   -1   0
 $EndComp
+$Comp
+L DIODE D?
+U 1 1 51BE5B9A
+P -50 7800
+F 0 "D?" H -150 7750 40  0000 C CNN
+F 1 "DIODE" H -50 7850 40  0000 C CNN
+F 2 "~" H -50 7800 60  0000 C CNN
+F 3 "~" H -50 7800 60  0000 C CNN
+	1    -50  7800
+	1    0    0    -1
+$EndComp
 Wire Wire Line
 	5850 5300 8650 5300
@@
 	9400 -1800 9400 -2350
 Wire Wire Line
-	9400 -2350 10400 -2350
-Wire Wire Line
 	9500 -1800 9500 -2350
 Connection ~ 9500 -2350
@@
 Connection ~ 10300 -2350
 Wire Wire Line
-	10400 -3000 10400 -1800
-Connection ~ 10400 -2350
-Wire Wire Line
 	7450 4450 7450 4550
 Wire Wire Line
@@
 Connection ~ 600  1550
 Wire Wire Line
-	11700 6050 -1050 6050
+	-1650 6050 11700 6050
 Connection ~ 7600 4550
 Wire Wire Line
@@
 Connection ~ 9400 -2350
 Wire Wire Line
-	-1050 6050 -1050 6900
-Wire Wire Line
 	600  6050 600  1550
-Connection ~ -1050 6900
-Connection ~ -650 7500
-Wire Wire Line
-	9350 -3400 21950 -3400
-Wire Wire Line
-	-650 7850 -650 7500
-Wire Wire Line
-	-650 8250 -650 13300
-Connection ~ -650 8250
-Connection ~ -650 7850
-Wire Wire Line
-	9350 -3400 9350 -3000
-Wire Wire Line
-	9350 -3000 9650 -3000
-Connection ~ 9650 -3000
-Wire Wire Line
-	10400 -3000 10150 -3000
-Connection ~ 10150 -3000
 Connection ~ 9400 -1300
 Connection ~ 9500 -1300
@@
 	14700 4050 14700 -1000
 Wire Wire Line
-	17600 7700 16800 7700
-Wire Wire Line
-	16800 7700 16800 -2800
+	16800 7700 17600 7700
 Wire Wire Line
-	16800 -2800 10150 -2800
-Connection ~ 10150 -2800
+	16800 -3150 16800 7700
 Connection ~ 17600 7700
 Connection ~ 17600 7900
@@
 	16000 8900 17600 8900
 Wire Wire Line
-	21950 -3400 21950 8000
+	21950 -4350 21950 8000
 Wire Wire Line
 	21950 8000 20300 8000
@@
 	21150 7700 21150 13300
 Wire Wire Line
-	21150 13300 -650 13300
+	21150 13300 -1650 13300
 Wire Wire Line
 	17600 8700 17200 8700
@@
 Connection ~ 17600 8800
 Connection ~ 20300 7700
-$Comp
-L USB-MINI-B CON1
-U 1 1 51BB5678
-P 5000 -2300
-F 0 "CON1" H 4750 -1850 60  0000 C CNN
-F 1 "USB-MINI-B" H 4950 -2800 60  0000 C CNN
-F 2 "" H 5000 -2300 60  0000 C CNN
-F 3 "" H 5000 -2300 60  0000 C CNN
-	1    5000 -2300
-	1    0    0    -1
-$EndComp
-Text Label 17600 7700 2    60   ~ 0
-GND
-$Comp
-L USB-MINI-B_EXT U1
-U 1 1 51BB56F7
-P 3600 -2300
-F 0 "U1" H 3600 -1850 60  0000 C CNN
-F 1 "USB-MINI-B_EXT" H 3600 -2800 60  0000 C CNN
-F 2 "" H 3600 -2300 60  0000 C CNN
-F 3 "" H 3600 -2300 60  0000 C CNN
-	1    3600 -2300
-	1    0    0    -1
-$EndComp
 Wire Wire Line
 	4050 -2600 4450 -2600
@@
 Connection ~ 4050 -2150
 Connection ~ 4050 -2000
+Connection ~ 10200 -3150
+Connection ~ 9500 -3150
+Connection ~ 9850 -3600
+Wire Wire Line
+	9850 -3600 9850 -4350
+Wire Wire Line
+	9850 -4350 21950 -4350
+Wire Wire Line
+	-1650 13300 -1650 11100
+Connection ~ -1650 11100
+Connection ~ -1650 10700
+Wire Wire Line
+	-1650 10700 -1650 10100
+Connection ~ -1650 10100
+Wire Wire Line
+	-2500 8900 -3400 8900
+Connection ~ -2500 8900
+Connection ~ -2500 9000
+Connection ~ -3400 8900
+Connection ~ -4000 8900
+Connection ~ -3250 9000
+Connection ~ -2750 9000
+Wire Wire Line
+	-2500 9000 -2750 9000
+Wire Wire Line
+	-4000 8900 -4250 8900
+Wire Wire Line
+	-4250 9000 -3250 9000
+Wire Wire Line
+	-800 8650 -350 8650
+Connection ~ -350 8650
+Connection ~ -800 8650
+Connection ~ 50   8650
+Wire Wire Line
+	-1650 6050 -1650 6500
+Wire Wire Line
+	10300 -2350 9150 -2350
+Wire Wire Line
+	9150 -2350 9150 -3150
+Wire Wire Line
+	9150 -3150 9500 -3150
+Wire Wire Line
+	10200 -3150 16800 -3150
 $EndSCHEMATC

Commit message: Added GPL and killed some bogus cache files.
Parts:
- added C?: CP1, ~, symbol CP1
Connections:
- net GND: now also R?.2, VREG1.2 (Sw_Emit), C?.2
- net at VREG1.5 (V_Sense): now also R?.1, R?.2
- net at VREG1.6 (VCC): now also C?.1, R?.1
- net at VREG1.7 (I_Sense): now also D?.1 (A), L?.1, R?.1, R?.2
- net at C?.1: now also D?.2 (K), R?.1
Other:
- moved on the sheet: D?, R?
Changed lines of the file:
@@
-EESchema Schematic File Version 2  date 16/06/2013 8:00:48 PM
+EESchema Schematic File Version 2  date 20/06/2013 6:29:09 PM
 LIBS:components
 LIBS:toasty-tkl-cache
@@
 Sheet 1 1
 Title "Toasty TKL"
-Date "17 jun 2013"
+Date "21 jun 2013"
 Rev "REV 1A"
 Comp ""
@@
 L RESISTOR R?
 U 1 1 51BE5B5E
-P 0 10000
-F 0 "R?" V 0   9900 50  0000 C CNN
-F 1 "RESISTOR" V 0   10100 50  0000 C CNN
-F 2 "~" H 0   10000 60  0000 C CNN
-F 3 "~" H 0   10000 60  0000 C CNN
-	1    0    10000
-	1    0    0    -1
+P -900 9500
+F 0 "R?" V -900 9400 50  0000 C CNN
+F 1 "RESISTOR" V -900 9600 50  0000 C CNN
+F 2 "~" H -900 9500 60  0000 C CNN
+F 3 "~" H -900 9500 60  0000 C CNN
+	1    -900 9500
+	0    -1   -1   0
 $EndComp
 $Comp
 L RESISTOR R?
 U 1 1 51BE5B6D
-P 250 10000
-F 0 "R?" V 250 9900 50  0000 C CNN
-F 1 "RESISTOR" V 250 10100 50  0000 C CNN
-F 2 "~" H 250 10000 60  0000 C CNN
-F 3 "~" H 250 10000 60  0000 C CNN
-	1    250  10000
-	1    0    0    -1
+P -3650 8600
+F 0 "R?" V -3650 8500 50  0000 C CNN
+F 1 "RESISTOR" V -3650 8700 50  0000 C CNN
+F 2 "~" H -3650 8600 60  0000 C CNN
+F 3 "~" H -3650 8600 60  0000 C CNN
+	1    -3650 8600
+	0    -1   -1   0
 $EndComp
 $Comp
 L RESISTOR R?
 U 1 1 51BE5B7C
-P 500 10000
-F 0 "R?" V 500 9900 50  0000 C CNN
-F 1 "RESISTOR" V 500 10100 50  0000 C CNN
-F 2 "~" H 500 10000 60  0000 C CNN
-F 3 "~" H 500 10000 60  0000 C CNN
-	1    500  10000
-	1    0    0    -1
+P -850 11550
+F 0 "R?" V -850 11450 50  0000 C CNN
+F 1 "RESISTOR" V -850 11650 50  0000 C CNN
+F 2 "~" H -850 11550 60  0000 C CNN
+F 3 "~" H -850 11550 60  0000 C CNN
+	1    -850 11550
+	0    -1   -1   0
 $EndComp
 $Comp
@@
 L DIODE D?
 U 1 1 51BE5B9A
-P -50 7800
-F 0 "D?" H -150 7750 40  0000 C CNN
-F 1 "DIODE" H -50 7850 40  0000 C CNN
-F 2 "~" H -50 7800 60  0000 C CNN
-F 3 "~" H -50 7800 60  0000 C CNN
-	1    -50  7800
-	1    0    0    -1
+P -1650 7400
+F 0 "D?" H -1750 7350 40  0000 C CNN
+F 1 "DIODE" H -1650 7450 40  0000 C CNN
+F 2 "~" H -1650 7400 60  0000 C CNN
+F 3 "~" H -1650 7400 60  0000 C CNN
+	1    -1650 7400
+	0    -1   -1   0
 $EndComp
 Wire Wire Line
@@
 Wire Wire Line
 	10200 -3150 16800 -3150
+Wire Wire Line
+	-1650 9700 -1650 9300
+Connection ~ -1650 9700
+Connection ~ -1650 9300
+Wire Wire Line
+	-1650 9500 -1150 9500
+Connection ~ -1650 9500
+Wire Wire Line
+	-650 9500 -400 9500
+Wire Wire Line
+	-400 8950 -400 10300
+Wire Wire Line
+	-400 8950 -800 8950
+Connection ~ -650 9500
+Connection ~ -1150 9500
+Connection ~ -800 8950
+Connection ~ -400 9500
+Wire Wire Line
+	-4250 7750 -4250 10300
+Wire Wire Line
+	-4250 10300 -400 10300
+Connection ~ -4250 9000
+Wire Wire Line
+	-4250 7750 -1650 7750
+Wire Wire Line
+	-1650 7750 -1650 7600
+Connection ~ -4250 8900
+Wire Wire Line
+	-1650 7200 -1650 6900
+Connection ~ -1650 6900
+Connection ~ -1650 7200
+Wire Wire Line
+	-2500 8600 -3400 8600
+Wire Wire Line
+	-3900 8600 -4750 8600
+Wire Wire Line
+	-4750 8600 -4750 7050
+Wire Wire Line
+	-4750 7050 -1650 7050
+Connection ~ -1650 7050
+Connection ~ -3900 8600
+Connection ~ -3400 8600
+Wire Wire Line
+	0    14150 16500 14150
+Wire Wire Line
+	16500 14150 16500 7500
+Wire Wire Line
+	16500 7500 16800 7500
+Connection ~ 16800 7500
+$Comp
+L CP1 C?
+U 1 1 51C3F6C2
+P 0 10500
+F 0 "C?" H 50  10600 50  0000 L CNN
+F 1 "CP1" H 50  10400 50  0000 L CNN
+F 2 "~" H 0   10500 60  0000 C CNN
+F 3 "~" H 0   10500 60  0000 C CNN
+	1    0    10500
+	1    0    0    -1
+$EndComp
+Wire Wire Line
+	-3000 8600 -3000 11550
+Connection ~ -3000 8600
+Wire Wire Line
+	-3000 11550 -1100 11550
+Wire Wire Line
+	-600 11550 0    11550
+Wire Wire Line
+	0    10700 0    14150
+Connection ~ 0    11550
+Wire Wire Line
+	-2500 8750 -4550 8750
+Wire Wire Line
+	-4550 8750 -4550 11800
+Wire Wire Line
+	-4550 11800 0    11800
+Connection ~ 0    11800
 $EndSCHEMATC

Commit message: Updates to kicad files.  Added DXF plot altered for water jet shop.
Parts:
- removed C?: CP1, ~, symbol CP1
- gave numbers to parts that had none: 10
Connections:
- net GND: now also C1.2, Ct1.2, VREG1.4 (GND)
- net LEDCOL0: now also BCR2.1, Co1.1, D2.2 (K)
- net at C1.1, Rsc1.1, VREG1.6 (VCC): now also F1.1
Other:
- moved on the sheet: C1, Ct1, F1
Changed lines of the file:
@@
-EESchema Schematic File Version 2  date 20/06/2013 6:29:09 PM
+EESchema Schematic File Version 2  date 23/06/2013 4:53:48 PM
 LIBS:components
 LIBS:toasty-tkl-cache
@@
 Sheet 1 1
 Title "Toasty TKL"
-Date "21 jun 2013"
+Date "23 jun 2013"
 Rev "REV 1A"
 Comp ""
@@
 L FUSE F1
 U 1 1 519CE3F5
-P -1650 10900
-F 0 "F1" H -1650 10750 60  0000 C CNN
-F 1 "FUSE" H -1650 11050 60  0000 C CNN
-F 2 "" H -1650 10900 60  0000 C CNN
-F 3 "" H -1650 10900 60  0000 C CNN
-	1    -1650 10900
+P -2050 12600
+F 0 "F1" H -2050 12450 60  0000 C CNN
+F 1 "FUSE" H -2050 12750 60  0000 C CNN
+F 2 "" H -2050 12600 60  0000 C CNN
+F 3 "" H -2050 12600 60  0000 C CNN
+	1    -2050 12600
 	0    -1   -1   0
 $EndComp
@@
 $EndComp
 $Comp
-L FET_N Q?
+L FET_N Q1
 U 1 1 51BE4888
 P 9850 -3300
-F 0 "Q?" H 9753 -3050 70  0000 C CNN
+F 0 "Q1" H 9753 -3050 70  0000 C CNN
 F 1 "FET_N" H 9703 -3547 60  0000 C CNN
 F 2 "~" H 9850 -3300 60  0000 C CNN
@@
 $EndComp
 $Comp
-L CP1 C?
-U 1 1 51BE5B22
-P -1650 6700
-F 0 "C?" H -1600 6800 50  0000 L CNN
-F 1 "CP1" H -1600 6600 50  0000 L CNN
-F 2 "~" H -1650 6700 60  0000 C CNN
-F 3 "~" H -1650 6700 60  0000 C CNN
-	1    -1650 6700
-	-1   0    0    1
-$EndComp
-$Comp
-L CP1 C?
+L CP1 C1
 U 1 1 51BE5B31
-P -1650 9900
-F 0 "C?" H -1600 10000 50  0000 L CNN
-F 1 "CP1" H -1600 9800 50  0000 L CNN
-F 2 "~" H -1650 9900 60  0000 C CNN
-F 3 "~" H -1650 9900 60  0000 C CNN
-	1    -1650 9900
+P -1650 10800
+F 0 "C1" H -1600 10900 50  0000 L CNN
+F 1 "CP1" H -1600 10700 50  0000 L CNN
+F 2 "~" H -1650 10800 60  0000 C CNN
+F 3 "~" H -1650 10800 60  0000 C CNN
+	1    -1650 10800
 	1    0    0    -1
 $EndComp
 $Comp
-L CP1 C?
+L CP1 Ct1
 U 1 1 51BE5B40
-P -150 8650
-F 0 "C?" H -100 8750 50  0000 L CNN
-F 1 "CP1" H -100 8550 50  0000 L CNN
-F 2 "~" H -150 8650 60  0000 C CNN
-F 3 "~" H -150 8650 60  0000 C CNN
-	1    -150 8650
+P -450 8650
+F 0 "Ct1" H -400 8750 50  0000 L CNN
+F 1 "CP1" H -400 8550 50  0000 L CNN
+F 2 "~" H -450 8650 60  0000 C CNN
+F 3 "~" H -450 8650 60  0000 C CNN
+	1    -450 8650
 	0    -1   -1   0
 $EndComp
 $Comp
-L RESISTOR R?
+L RESISTOR BCR0
 U 1 1 51BE5B4F
 P -3000 9000
-F 0 "R?" V -3000 8900 50  0000 C CNN
-F 1 "RESISTOR" V -3000 9100 50  0000 C CNN
+F 0 "BCR0" V -3100 9000 50  0000 C CNN
+F 1 "RESISTOR" V -3000 9000 50  0000 C CNN
 F 2 "~" H -3000 9000 60  0000 C CNN
 F 3 "~" H -3000 9000 60  0000 C CNN
@@
 $EndComp
 $Comp
-L RESISTOR R?
+L RESISTOR Rsc1
 U 1 1 51BE5B5E
 P -900 9500
-F 0 "R?" V -900 9400 50  0000 C CNN
-F 1 "RESISTOR" V -900 9600 50  0000 C CNN
+F 0 "Rsc1" V -800 9500 50  0000 C CNN
+F 1 "RESISTOR" V -900 9500 50  0000 C CNN
 F 2 "~" H -900 9500 60  0000 C CNN
 F 3 "~" H -900 9500 60  0000 C CNN
@@
 $EndComp
 $Comp
-L RESISTOR R?
+L RESISTOR BCR2
 U 1 1 51BE5B6D
 P -3650 8600
-F 0 "R?" V -3650 8500 50  0000 C CNN
-F 1 "RESISTOR" V -3650 8700 50  0000 C CNN
+F 0 "BCR2" V -3550 8600 50  0000 C CNN
+F 1 "RESISTOR" V -3650 8600 50  0000 C CNN
 F 2 "~" H -3650 8600 60  0000 C CNN
 F 3 "~" H -3650 8600 60  0000 C CNN
@@
 $EndComp
 $Comp
-L RESISTOR R?
+L RESISTOR BCR1
 U 1 1 51BE5B7C
 P -850 11550
-F 0 "R?" V -850 11450 50  0000 C CNN
-F 1 "RESISTOR" V -850 11650 50  0000 C CNN
+F 0 "BCR1" V -750 11550 50  0000 C CNN
+F 1 "RESISTOR" V -850 11550 50  0000 C CNN
 F 2 "~" H -850 11550 60  0000 C CNN
 F 3 "~" H -850 11550 60  0000 C CNN
@@
 $EndComp
 $Comp
-L INDUCTOR L?
+L INDUCTOR L1
 U 1 1 51BE5B8B
 P -3700 8900
-F 0 "L?" V -3750 8900 40  0000 C CNN
+F 0 "L1" V -3750 8900 40  0000 C CNN
 F 1 "INDUCTOR" V -3600 8900 40  0000 C CNN
 F 2 "~" H -3700 8900 60  0000 C CNN
@@
 $EndComp
 $Comp
-L DIODE D?
+L DIODE D2
 U 1 1 51BE5B9A
 P -1650 7400
-F 0 "D?" H -1750 7350 40  0000 C CNN
+F 0 "D2" H -1750 7350 40  0000 C CNN
 F 1 "DIODE" H -1650 7450 40  0000 C CNN
 F 2 "~" H -1650 7400 60  0000 C CNN
@@
 	0    -1   -1   0
 $EndComp
+$Comp
+L CP1 Co1
+U 1 1 51C3F6C2
+P 0 10500
+F 0 "Co1" H 50  10600 50  0000 L CNN
+F 1 "CP1" H 50  10400 50  0000 L CNN
+F 2 "~" H 0   10500 60  0000 C CNN
+F 3 "~" H 0   10500 60  0000 C CNN
+	1    0    10500
+	1    0    0    -1
+$EndComp
 Wire Wire Line
 	5850 5300 8650 5300
@@
 	21150 7700 21150 13300
 Wire Wire Line
-	21150 13300 -1650 13300
+	21150 13300 -2050 13300
 Wire Wire Line
 	17600 8700 17200 8700
@@
 	9850 -4350 21950 -4350
 Wire Wire Line
-	-1650 13300 -1650 11100
-Connection ~ -1650 11100
-Connection ~ -1650 10700
-Wire Wire Line
-	-1650 10700 -1650 10100
-Connection ~ -1650 10100
-Wire Wire Line
 	-2500 8900 -3400 8900
 Connection ~ -2500 8900
@@
 Wire Wire Line
 	-4250 9000 -3250 9000
-Wire Wire Line
-	-800 8650 -350 8650
-Connection ~ -350 8650
 Connection ~ -800 8650
-Connection ~ 50   8650
-Wire Wire Line
-	-1650 6050 -1650 6500
 Wire Wire Line
 	10300 -2350 9150 -2350
@@
 Wire Wire Line
 	10200 -3150 16800 -3150
-Wire Wire Line
-	-1650 9700 -1650 9300
-Connection ~ -1650 9700
 Connection ~ -1650 9300
 Wire Wire Line
-	-1650 9500 -1150 9500
+	-2050 9500 -1150 9500
 Connection ~ -1650 9500
 Wire Wire Line
 	-650 9500 -400 9500
 Wire Wire Line
-	-400 8950 -400 10300
-Wire Wire Line
 	-400 8950 -800 8950
 Connection ~ -650 9500
@@
 Connection ~ -800 8950
 Connection ~ -400 9500
-Wire Wire Line
-	-4250 7750 -4250 10300
-Wire Wire Line
-	-4250 10300 -400 10300
 Connection ~ -4250 9000
 Wire Wire Line
@@
 Connection ~ -4250 8900
 Wire Wire Line
-	-1650 7200 -1650 6900
-Connection ~ -1650 6900
+	-1650 6050 -1650 7200
 Connection ~ -1650 7200
 Wire Wire Line
 	-2500 8600 -3400 8600
-Wire Wire Line
-	-3900 8600 -4750 8600
-Wire Wire Line
-	-4750 8600 -4750 7050
-Wire Wire Line
-	-4750 7050 -1650 7050
 Connection ~ -1650 7050
 Connection ~ -3900 8600
@@
 	16500 7500 16800 7500
 Connection ~ 16800 7500
-$Comp
-L CP1 C?
-U 1 1 51C3F6C2
-P 0 10500
-F 0 "C?" H 50  10600 50  0000 L CNN
-F 1 "CP1" H 50  10400 50  0000 L CNN
-F 2 "~" H 0   10500 60  0000 C CNN
-F 3 "~" H 0   10500 60  0000 C CNN
-	1    0    10500
-	1    0    0    -1
-$EndComp
 Wire Wire Line
 	-3000 8600 -3000 11550
@@
 	-3000 11550 -1100 11550
 Wire Wire Line
-	-600 11550 0    11550
+	-600 11550 500  11550
 Wire Wire Line
 	0    10700 0    14150
@@
 	-4550 11800 0    11800
 Connection ~ 0    11800
+Connection ~ -2500 8750
+Connection ~ -2500 8600
+Connection ~ -600 11550
+Connection ~ -1100 11550
+Connection ~ 0    10700
+Connection ~ -1650 7600
+Connection ~ 0    10300
+Connection ~ -1650 8300
+Wire Wire Line
+	-1650 8300 -1650 7950
+Wire Wire Line
+	-1650 7950 500  7950
+Wire Wire Line
+	500  7950 500  11550
+Wire Wire Line
+	-1650 11200 300  11200
+Connection ~ 0    11200
+Wire Wire Line
+	-2050 9500 -2050 12400
+Wire Wire Line
+	-1650 9300 -1650 10600
+Wire Wire Line
+	-2050 13300 -2050 12800
+Wire Wire Line
+	-1650 11000 -1650 11200
+Wire Wire Line
+	-4250 7750 -4250 9950
+Wire Wire Line
+	-4250 9950 -400 9950
+Wire Wire Line
+	-400 9950 -400 8950
+Wire Wire Line
+	-800 8650 -650 8650
+Wire Wire Line
+	-250 8650 300  8650
+Wire Wire Line
+	0    7050 0    10300
+Wire Wire Line
+	300  8650 300  11200
+Wire Wire Line
+	-3900 8600 -4550 8600
+Wire Wire Line
+	-4550 8600 -4550 7050
+Wire Wire Line
+	-4550 7050 0    7050
+Connection ~ -250 8650
+Connection ~ -1650 11000
+Connection ~ -1650 10600
+Connection ~ -2050 12400
+Connection ~ -2050 12800
+Connection ~ -650 8650
 $EndSCHEMATC
