File: kicad_files/toasty-tkl.sch (KiCad schematic (older format))
At the start: 204 parts, among them CON1 USB-MINI-B, Q1 FET_N, SW0:0 ESC, SW0:10 F9, SW0:11 F10, SW0:12 F11, SW0:13 F12, SW0:14 PRINT, SW0:15 SCROLL LOCK, SW0:2 F1, SW0:3 F2, SW0:4 F3, SW0:5 F4, SW0:6 F5, SW0:7 F6, SW0:8 F7, SW0:9 F8, SW1:0 `, SW1:1 1, SW1:10 0, SW1:11 -, SW1:12 =, SW1:13 BACK SPACE, SW1:14 INSERT, SW1:15 HOME, SW1:2 2, SW1:3 3, SW1:4 4, SW1:5 5, SW1:6 6, SW1:7 7, SW1:8 8, SW1:9 9, SW2:0 TAB, SW2:1 Q, SW2:10 P, SW2:11 [, SW2:12 ], SW2:13 \\, SW2:14 DELETE, SW2:15 END, SW2:2 W, SW2:3 E, SW2:4 R, SW2:5 T, SW2:6 Y, SW2:7 U, SW2:8 I, SW2:9 O, SW3:0 CAPS LOCK, SW3:1 A, SW3:10 ;, SW3:11 ', SW3:13 ENTER, SW3:14 PAGE UP, SW3:15 PAUSE, SW3:2 S, SW3:3 D, SW3:4 F, SW3:5 G, SW3:6 H, SW3:7 J, SW3:8 K, SW3:9 L, SW4:0 LEFT SHIFT, SW4:1 Z, SW4:10 /, SW4:13 RIGHT SHIFT, SW4:14 PAGE DOWN, SW4:15 UP, SW4:2 X, SW4:3 C, SW4:4 V, SW4:5 B, SW4:6 N, SW4:7 M, SW4:8 ,, SW4:9 ., SW5:0 LEFT CTRL, SW5:1 LEFT WINDOWS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

Commit message: Removed unnecesarry joints, added values for parts in schema.  Fixed traces.
Parts:
- BC_Co1: value CP1 -> 47µF
- BC_Ct1: value CP1 -> 1000pF
- BC_Cvcc1: value CP1 -> 100µF
- BC_D1: value DIODE -> 30V 1A
- BC_F1: value FUSE -> .750A 125V
- BC_L1: value INDUCTOR -> 100µH
- BC_R0, R0, R1, R2, R3, R4, R5, R6, R7, R8, R9: value RESISTOR -> 180 OHM 1/8W
- BC_R1: value RESISTOR -> 3.6K OHM 1/8W
- BC_R2: value RESISTOR -> 51K OHM 1/8W
- BC_Rsc1: value RESISTOR -> 0.33 OHM 1/2W
- D0, D1: value LED -> 2.2V 20mA
- LED_R0, LED_R1: value RESISTOR -> 2.7K OHM 1/8W
- Q1: value FET_N -> 60V 1.2A
- R10: value RESISTOR -> 510 OHM 1/8W
Connections:
- net COL 7: no longer D1:7.1 (A)

Commit message: Rewired PD6 pin on teensy, it wouldn't work as a column pin.  LED is present on the line.
Connections:
- net COL 0: now also U0.45 (PB0); no longer U0.33 (PF7)
- net COL 1: now also U0.46 (PB1); no longer U0.34 (PF6)
- net COL 10: now also U0.38 (PF2); no longer U0.8 (PD5)
- net COL 11: now also U0.37 (PF3); no longer U0.7 (PD4)
- net COL 12: now also U0.36 (PF4); no longer U0.6 (PD3)
- net COL 13: now also U0.35 (PF5); no longer U0.5 (PD2)
- net COL 14: now also U0.34 (PF6); no longer U0.4 (PD1)
- net COL 15: now also U0.33 (PF7); no longer U0.3 (PD0)
- net COL 2: now also U0.47 (PB2); no longer U0.35 (PF5)
- net COL 3: now also U0.48 (PB3); no longer U0.36 (PF4)
- net COL 4: now also U0.49 (PB4); no longer U0.37 (PF3)
- net COL 5: now also U0.50 (PB5); no longer U0.38 (PF2)
- net COL 6: now also U0.51 (PB6); no longer U0.39 (PF1)
- net COL 7: now also U0.2 (PB7); no longer U0.40 (PF0)
- net COL 8: now also U0.40 (PF0); no longer U0.10 (PD7)
- net COL 9: now also U0.39 (PF1); no longer U0.9 (PD6)
- net LED 0: now also U0.18 (PC5); no longer U0.2 (PB7)
- net ROW 5: now also U0.20 (PC7); no longer U0.18 (PC5)
- net Q1: now reaches Q1.1 (G)
- net Q1: now also U0.4 (PD1); no longer U0.49 (PB4)

Commit message: Fixed some traces.  Added more silk screen text.
Connections:
- net COL 7: now also D1:7.1 (A)
Changed lines of the file:
@@
 Wire Wire Line
 	9850 -4350 17000 -4350
+Connection ~ 6850 2450
 $EndSCHEMATC
