File: kicad_files/toasty-tkl.kicad_pcb (KiCad board)
At the start: 2 copper layers, 345.7 x 134.1 mm, 204 parts, among them CON1 USB-MINI-B, Q1 60V 1.2A, SW0:0 ESC, SW0:10 F9, SW0:11 F10, SW0:12 F11, SW0:13 F12, SW0:14 PRINT, SW0:15 SCROLL LOCK, SW0:2 F1, SW0:3 F2, SW0:4 F3, SW0:5 F4, SW0:6 F5, SW0:7 F6, SW0:8 F7, SW0:9 F8, SW1:0 `, SW1:1 1, SW1:10 0, SW1:11 -, SW1:12 =, SW1:13 BACK SPACE, SW1:14 INSERT, SW1:15 HOME, SW1:2 2, SW1:3 3, SW1:4 4, SW1:5 5, SW1:6 6, SW1:7 7, SW1:8 8, SW1:9 9, SW2:0 TAB, SW2:1 Q, SW2:10 P, SW2:11 [, SW2:12 ], SW2:13 \, SW2:14 DELETE, SW2:15 END, SW2:2 W, SW2:3 E, SW2:4 R, SW2:5 T, SW2:6 Y, SW2:7 U, SW2:8 I, SW2:9 O, SW3:0 CAPS LOCK, SW3:1 A, SW3:10 ;, SW3:11 ', SW3:13 ENTER, SW3:14 PAGE UP, SW3:15 PAUSE, SW3:2 S, SW3:3 D, SW3:4 F, SW3:5 G, SW3:6 H, SW3:7 J, SW3:8 K, SW3:9 L, SW4:0 LEFT SHIFT, SW4:1 Z, SW4:10 /, SW4:13 RIGHT SHIFT, SW4:14 PAGE DOWN, SW4:15 UP, SW4:2 X, SW4:3 C, SW4:4 V, SW4:5 B, SW4:6 N, SW4:7 M, SW4:8 ,, SW4:9 ., SW5:0 LEFT CTRL, SW5:1 LEFT WINDOWS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

Commit message: did a couple trace changes
Routing:
- net /LEDROW6: track 45.5 -> 49.0 mm
- net /LED 0: track 69.2 -> 67.9 mm
Other:
- board text added: "USB MINI-B"
- board text removed: "USB-MINI-B"
Changed lines of the file:
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@@
-(kicad_pcb (version 3) (host pcbnew "(2013-05-31 BZR 4019)-stable")
+(kicad_pcb (version 3) (host pcbnew "(2013-04-19 BZR 4011)-stable")
   (general
     (links 408)
@@
       (usegerberextensions false)
       (excludeedgelayer true)
-      (linewidth 0.150000)
+      (linewidth 0)
       (plotframeref false)
       (viasonmask false)
@@
     (effects (font (size 0.762 0.762) (thickness 0.1778)) (justify mirror))
   )
-  (gr_text USB-MINI-B (at 191.262 7.874) (layer B.SilkS)
-    (effects (font (size 0.4572 0.4572) (thickness 0.0762)) (justify mirror))
+  (gr_text "USB\nMINI-B" (at 191.262 7.874) (layer B.SilkS)
+    (effects (font (size 0.5588 0.5588) (thickness 0.0762)) (justify mirror))
   )
   (gr_text "BC_R1: 3.6K OHM 1/8W" (at 202.565 125.6665) (layer B.SilkS)
@@
   (segment (start 284.226 31.242) (end 284.226 33.782) (width 0.254) (layer B.Cu) (net 6) (status 10))
   (segment (start 284.226 33.782) (end 284.226 38.862) (width 0.254) (layer B.Cu) (net 6))
+  (segment (start 271.145 32.893) (end 294.767 32.893) (width 0.254) (layer F.Cu) (net 7))
   (segment (start 303.276 52.578) (end 303.276 84.328) (width 0.254) (layer B.Cu) (net 7))
   (segment (start 304.546 88.138) (end 307.594 88.138) (width 0.254) (layer F.Cu) (net 7))
@@
   (via (at 272.796 116.586) (size 0.889) (layers F.Cu B.Cu) (net 7))
   (segment (start 272.796 116.586) (end 269.494 113.284) (width 0.254) (layer B.Cu) (net 7))
-  (segment (start 271.272 32.766) (end 294.64 32.766) (width 0.254) (layer F.Cu) (net 7))
-  (segment (start 297.688 35.814) (end 294.64 32.766) (width 0.254) (layer F.Cu) (net 7))
+  (segment (start 297.688 35.814) (end 294.767 32.893) (width 0.254) (layer F.Cu) (net 7))
   (segment (start 269.494 106.68) (end 272.034 104.14) (width 0.254) (layer B.Cu) (net 7))
   (segment (start 272.034 104.14) (end 272.034 68.834) (width 0.254) (layer B.Cu) (net 7))
@@
   (segment (start 269.24 34.798) (end 270.256 33.782) (width 0.254) (layer B.Cu) (net 7))
   (via (at 270.256 33.782) (size 0.889) (layers F.Cu B.Cu) (net 7))
-  (segment (start 270.256 33.782) (end 271.272 32.766) (width 0.254) (layer F.Cu) (net 7))
+  (segment (start 270.256 33.782) (end 271.145 32.893) (width 0.254) (layer F.Cu) (net 7))
   (segment (start 269.494 113.284) (end 269.494 106.68) (width 0.254) (layer B.Cu) (net 7))
   (segment (start 321.31 64.516) (end 324.612 61.214) (width 0.254) (layer B.Cu) (net 7) (status 10))
@@
   (segment (start 319.532 107.87126) (end 319.70726 107.87126) (width 0.508) (layer B.Cu) (net 17))
   (segment (start 319.70726 107.87126) (end 322.072 110.236) (width 0.508) (layer B.Cu) (net 17))
+  (segment (start 343.662 51.308) (end 341.376 49.022) (width 0.508) (layer B.Cu) (net 18))
+  (segment (start 343.662 72.39) (end 343.662 51.308) (width 0.508) (layer B.Cu) (net 18))
   (segment (start 341.63 82.804) (end 354.838 82.804) (width 0.508) (layer F.Cu) (net 18))
   (segment (start 343.662 72.39) (end 343.662 75.057) (width 0.508) (layer B.Cu) (net 18))
-  (segment (start 342.011 70.739) (end 343.662 72.39) (width 0.508) (layer B.Cu) (net 18))
   (segment (start 330.835 40.513) (end 336.677 40.513) (width 0.508) (layer F.Cu) (net 18))
-  (segment (start 337.566 41.402) (end 336.677 40.513) (width 0.508) (layer F.Cu) (net 18))
-  (via (at 337.566 41.402) (size 0.889) (layers F.Cu B.Cu) (net 18))
-  (segment (start 341.376 49.022) (end 338.328 45.974) (width 0.508) (layer B.Cu) (net 18))
-  (segment (start 338.328 42.164) (end 337.566 41.402) (width 0.508) (layer B.Cu) (net 18))
   (segment (start 338.328 45.974) (end 338.328 42.164) (width 0.508) (layer B.Cu) (net 18))
-  (segment (start 341.376 51.054) (end 341.376 49.022) (width 0.508) (layer B.Cu) (net 18))
-  (segment (start 342.011 58.674) (end 339.852 56.515) (width 0.508) (layer B.Cu) (net 18))
-  (segment (start 339.852 56.515) (end 339.852 52.578) (width 0.508) (layer B.Cu) (net 18))
-  (segment (start 339.852 52.578) (end 341.376 51.054) (width 0.508) (layer B.Cu) (net 18))
-  (segment (start 342.011 70.739) (end 342.011 58.674) (width 0.508) (layer B.Cu) (net 18))
+  (segment (start 338.328 42.164) (end 337.566 41.402) (width 0.508) (layer B.Cu) (net 18))
+  (segment (start 341.376 49.022) (end 338.328 45.974) (width 0.508) (layer B.Cu) (net 18))
+  (via (at 337.566 41.402) (size 0.889) (layers F.Cu B.Cu) (net 18))
+  (segment (start 337.566 41.402) (end 336.677 40.513) (width 0.508) (layer F.Cu) (net 18))
   (via (at 341.63 82.804) (size 0.889) (layers F.Cu B.Cu) (net 18))
   (segment (start 341.63 77.089) (end 341.63 82.804) (width 0.508) (layer B.Cu) (net 18))
@@
   (segment (start 292.735 121.158) (end 298.1325 126.5555) (width 0.508) (layer B.Cu) (net 27))
   (segment (start 290.576 121.158) (end 292.735 121.158) (width 0.508) (layer B.Cu) (net 27) (status 10))
-  (segment (start 337.8454 59.9313) (end 337.8454 58.4454) (width 0.508) (layer F.Cu) (net 28))
-  (segment (start 337.312 57.912) (end 310.388 57.912) (width 0.508) (layer F.Cu) (net 28))
+  (segment (start 300.99 48.514) (end 304.038 51.562) (width 0.508) (layer B.Cu) (net 28))
+  (segment (start 300.99 45.466) (end 300.99 48.514) (width 0.508) (layer B.Cu) (net 28) (status 20))
   (segment (start 337.8454 58.4454) (end 337.312 57.912) (width 0.508) (layer F.Cu) (net 28))
+  (segment (start 337.312 57.912) (end 310.388 57.912) (width 0.508) (layer F.Cu) (net 28))
+  (segment (start 337.8454 58.4454) (end 337.8454 59.9313) (width 0.508) (layer F.Cu) (net 28))
+  (segment (start 304.546 57.912) (end 310.388 57.912) (width 0.508) (layer F.Cu) (net 28))
+  (via (at 304.546 57.912) (size 0.889) (layers F.Cu B.Cu) (net 28))
+  (segment (start 304.546 52.07) (end 304.546 57.912) (width 0.508) (layer B.Cu) (net 28))
+  (segment (start 304.292 51.816) (end 304.546 52.07) (width 0.508) (layer B.Cu) (net 28))
+  (segment (start 304.038 51.562) (end 304.292 51.816) (width 0.508) (layer B.Cu) (net 28))
   (segment (start 337.8454 59.9313) (end 337.8073 59.9313) (width 0.254) (layer F.Cu) (net 28) (status 30))
-  (segment (start 310.388 57.912) (end 300.99 48.514) (width 0.508) (layer F.Cu) (net 28))
-  (via (at 300.99 48.514) (size 0.889) (layers F.Cu B.Cu) (net 28))
-  (segment (start 300.99 48.514) (end 300.99 45.466) (width 0.508) (layer B.Cu) (net 28) (status 20))
   (segment (start 303.784 45.466) (end 303.784 48.514) (width 0.508) (layer B.Cu) (net 29))
   (segment (start 303.784 48.514) (end 307.467 52.197) (width 0.508) (layer B.Cu) (net 29))
@@
   (segment (start 358.648 78.74) (end 358.4067 78.9813) (width 0.508) (layer B.Cu) (net 211))
   (segment (start 358.4067 78.9813) (end 356.8954 78.9813) (width 0.508) (layer B.Cu) (net 211) (status 20))
+  (segment (start 346.202 134.366) (end 356.616 134.366) (width 0.508) (layer B.Cu) (net 212))
+  (segment (start 344.17 132.334) (end 346.202 134.366) (width 0.508) (layer B.Cu) (net 212))
+  (segment (start 344.17 132.334) (end 344.17 122.682) (width 0.508) (layer B.Cu) (net 212))
+  (segment (start 344.17 122.682) (end 341.376 119.888) (width 0.508) (layer B.Cu) (net 212))
   (segment (start 335.3054 118.491) (end 335.3054 118.5164) (width 0.508) (layer B.Cu) (net 212))
   (segment (start 341.35695 119.86895) (end 341.376 119.888) (width 0.508) (layer B.Cu) (net 212))
   (segment (start 335.3054 118.491) (end 335.3054 117.0813) (width 0.508) (layer B.Cu) (net 212) (status 20))
-  (segment (start 346.202 134.366) (end 356.616 134.366) (width 0.508) (layer B.Cu) (net 212))
   (segment (start 356.8954 136.1313) (end 356.8954 134.6454) (width 0.508) (layer B.Cu) (net 212) (status 20))
   (segment (start 356.616 134.366) (end 356.8954 134.6454) (width 0.508) (layer B.Cu) (net 212))
-  (segment (start 344.17 122.682) (end 341.376 119.888) (width 0.508) (layer B.Cu) (net 212))
-  (segment (start 344.17 132.334) (end 344.17 122.682) (width 0.508) (layer B.Cu) (net 212))
-  (segment (start 344.17 132.334) (end 346.202 134.366) (width 0.508) (layer B.Cu) (net 212))
   (segment (start 335.3054 118.5164) (end 336.296 119.507) (width 0.508) (layer B.Cu) (net 212))
   (segment (start 336.296 119.507) (end 340.995 119.507) (width 0.508) (layer B.Cu) (net 212))
