File: kicad_files/openclack-tkl.kicad_pcb (KiCad board)
At the start: 2 copper layers, 345.7 x 134.1 mm, 206 parts, among them CON1 USB-MINI-B, Q1 60V 1.2A, SW0:0 ESC, SW0:10 F9, SW0:11 F10, SW0:12 F11, SW0:13 F12, SW0:14 PRINT, SW0:15 SCROLL LOCK, SW0:2 F1, SW0:3 F2, SW0:4 F3, SW0:5 F4, SW0:6 F5, SW0:7 F6, SW0:8 F7, SW0:9 F8, SW1:0 `, SW1:1 1, SW1:10 0, SW1:11 -, SW1:12 =, SW1:13 BACK SPACE, SW1:14 INSERT, SW1:15 HOME, SW1:2 2, SW1:3 3, SW1:4 4, SW1:5 5, SW1:6 6, SW1:7 7, SW1:8 8, SW1:9 9, SW2:0 TAB, SW2:1 Q, SW2:10 P, SW2:11 [, SW2:12 ], SW2:13 \, SW2:14 DELETE, SW2:15 END, SW2:2 W, SW2:3 E, SW2:4 R, SW2:5 T, SW2:6 Y, SW2:7 U, SW2:8 I, SW2:9 O, SW3:0 CAPS LOCK, SW3:1 A, SW3:10 ;, SW3:11 ', SW3:13 ENTER, SW3:14 PAGE UP, SW3:15 PAUSE, SW3:2 S, SW3:3 D, SW3:4 F, SW3:5 G, SW3:6 H, SW3:7 J, SW3:8 K, SW3:9 L, SW4:0 LEFT SHIFT, SW4:1 Z, SW4:10 /, SW4:13 RIGHT SHIFT, SW4:14 PAGE DOWN, SW4:15 UP, SW4:2 X, SW4:3 C, SW4:4 V, SW4:5 B, SW4:6 N, SW4:7 M, SW4:8 ,, SW4:9 ., SW5:0 LEFT CTRL, SW5:1 LEFT WINDOWS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

Commit message: Fixed error for LED2 (scroll lock) gnd pin, found in prototype.
Routing:
- net /GND: track 179.1 -> 204.2 mm, vias 3 -> 5
Other:
- board text added: "LED_R1-2: 2.7K OHM 1/8W"
Changed lines of the file:
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@@
-(kicad_pcb (version 3) (host pcbnew "(2013-04-19 BZR 4011)-stable")
+(kicad_pcb (version 3) (host pcbnew "(2013-05-31 BZR 4019)-stable")
   (general
     (links 408)
-    (no_connects 1)
+    (no_connects 0)
     (area 3.963999 -151.103001 377.912301 568.094801)
     (thickness 1.6)
-    (drawings 297)
-    (tracks 1887)
+    (drawings 298)
+    (tracks 1897)
     (zones 0)
     (modules 206)
@@
     (22 B.Mask user)
     (23 F.Mask user)
-    (24 Dwgs.User user)
+    (24 Dwgs.User user hide)
     (25 Cmts.User user hide)
     (26 Eco1.User user hide)
@@
   )
   (setup
-    (last_trace_width 0.254)
+    (last_trace_width 0.508)
     (user_trace_width 0.508)
     (trace_clearance 0.254)
@@
       (usegerberextensions true)
       (excludeedgelayer true)
-      (linewidth 0)
+      (linewidth 0.150000)
       (plotframeref false)
       (viasonmask false)
@@
       (xy 4.83616 -2.4384) (xy 4.89204 -2.29108) (xy 4.89204 -2.29108)) (layer B.SilkS) (width 0.00254))
   )
-  (gr_text "Q1: 60V 1.2A" (at 204.343 137.922) (layer B.SilkS)
+  (gr_text "LED_R1-2: 2.7K OHM 1/8W" (at 198.501 119.507) (layer B.SilkS)
+    (effects (font (size 1.016 1.016) (thickness 0.1778)) (justify mirror))
+  )
+  (gr_text "Q1: 60V 1.2A" (at 204.216 138.43) (layer B.SilkS)
     (effects (font (size 1.016 1.016) (thickness 0.1778)) (justify mirror))
   )
@@
     (effects (font (size 1.016 1.016) (thickness 0.1778)) (justify mirror))
   )
-  (gr_text "BC_F1: .750A 125V" (at 202.057 136.525) (layer B.SilkS)
+  (gr_text "BC_F1: .750A 125V" (at 201.93 137.033) (layer B.SilkS)
     (effects (font (size 1.016 1.016) (thickness 0.1778)) (justify mirror))
   )
-  (gr_text "BC_D1: 30V 1A" (at 203.708 135.128) (layer B.SilkS)
+  (gr_text "BC_D1: 30V 1A" (at 203.581 135.636) (layer B.SilkS)
     (effects (font (size 1.016 1.016) (thickness 0.1778)) (justify mirror))
   )
-  (gr_text "BC_L1: 100µH" (at 203.962 133.731) (layer B.SilkS)
+  (gr_text "BC_L1: 100µH" (at 203.835 134.239) (layer B.SilkS)
     (effects (font (size 1.016 1.016) (thickness 0.1778)) (justify mirror))
   )
-  (gr_text "BC_Ct1: 1000pF" (at 203.327 132.334) (layer B.SilkS)
+  (gr_text "BC_Ct1: 1000pF" (at 203.2 132.842) (layer B.SilkS)
     (effects (font (size 1.016 1.016) (thickness 0.1778)) (justify mirror))
   )
-  (gr_text "BC_Cvcc1: 100µF" (at 202.819 130.937) (layer B.SilkS)
+  (gr_text "BC_Cvcc1: 100µF" (at 202.692 131.445) (layer B.SilkS)
     (effects (font (size 1.016 1.016) (thickness 0.1778)) (justify mirror))
   )
-  (gr_text "BC_Co1: 47µF" (at 204.089 129.54) (layer B.SilkS)
+  (gr_text "BC_Co1: 47µF" (at 203.962 130.048) (layer B.SilkS)
     (effects (font (size 1.016 1.016) (thickness 0.1778)) (justify mirror))
   )
-  (gr_text "BC_Rsc1: 0.33 OHM 1/2W" (at 199.39 128.143) (layer B.SilkS)
+  (gr_text "BC_Rsc1: 0.33 OHM 1/2W" (at 199.263 128.651) (layer B.SilkS)
     (effects (font (size 1.016 1.016) (thickness 0.1778)) (justify mirror))
   )
-  (gr_text "BC_R2: 51K OHM 1/8W" (at 200.406 126.619) (layer B.SilkS)
+  (gr_text "BC_R2: 51K OHM 1/8W" (at 200.279 127.127) (layer B.SilkS)
     (effects (font (size 1.016 1.016) (thickness 0.1778)) (justify mirror))
   )
-  (gr_text "BC_R0: 180 OHM 1/8W" (at 200.406 123.571) (layer B.SilkS)
+  (gr_text "BC_R0: 180 OHM 1/8W" (at 200.279 124.079) (layer B.SilkS)
     (effects (font (size 1.016 1.016) (thickness 0.1778)) (justify mirror))
   )
@@
     (effects (font (size 1.016 1.016) (thickness 0.1778)) (justify mirror))
   )
-  (gr_text "BC_R1: 3.6K OHM 1/8W" (at 200.152 125.095) (layer B.SilkS)
+  (gr_text "BC_R1: 3.6K OHM 1/8W" (at 200.025 125.603) (layer B.SilkS)
     (effects (font (size 1.016 1.016) (thickness 0.1778)) (justify mirror))
   )
-  (gr_text "R10: 510 OHM 1/8W" (at 201.295 122.047) (layer B.SilkS)
+  (gr_text "R10: 510 OHM 1/8W" (at 201.168 122.555) (layer B.SilkS)
     (effects (font (size 1.016 1.016) (thickness 0.1778)) (justify mirror))
   )
-  (gr_text "R0-9: 180 OHM 1/8W" (at 200.66 120.523) (layer B.SilkS)
+  (gr_text "R0-9: 180 OHM 1/8W" (at 200.533 121.031) (layer B.SilkS)
     (effects (font (size 1.016 1.016) (thickness 0.1778)) (justify mirror))
   )
@@
     (effects (font (size 1.5 1.5) (thickness 0.3)) (justify mirror))
   )
-  (gr_text "R ALT" (at 212.09 131.064 90) (layer B.SilkS)
+  (gr_text "R ALT" (at 211.963 130.937 90) (layer B.SilkS)
     (effects (font (size 1.5 1.5) (thickness 0.3)) (justify mirror))
   )
@@
   (via (at 292.608 45.72) (size 0.889) (layers F.Cu B.Cu) (net 16))
   (segment (start 292.608 48.26) (end 298.196 53.848) (width 0.254) (layer B.Cu) (net 16))
+  (segment (start 347.3704 40.5638) (end 347.3704 42.9006) (width 0.508) (layer B.Cu) (net 17))
+  (via (at 326.136 46.482) (size 0.889) (layers F.Cu B.Cu) (net 17))
+  (segment (start 328.676 46.482) (end 326.136 46.482) (width 0.508) (layer F.Cu) (net 17))
+  (segment (start 331.343 43.815) (end 328.676 46.482) (width 0.508) (layer F.Cu) (net 17))
+  (segment (start 337.185 43.815) (end 331.343 43.815) (width 0.508) (layer F.Cu) (net 17))
+  (segment (start 343.027 43.815) (end 337.185 43.815) (width 0.508) (layer F.Cu) (net 17))
+  (via (at 343.027 43.815) (size 0.889) (layers F.Cu B.Cu) (net 17))
+  (segment (start 346.456 43.815) (end 343.027 43.815) (width 0.508) (layer B.Cu) (net 17))
+  (segment (start 347.3704 42.9006) (end 346.456 43.815) (width 0.508) (layer B.Cu) (net 17))
   (segment (start 312.4454 85.3313) (end 312.4454 83.1596) (width 0.508) (layer B.Cu) (net 17))
   (segment (start 326.136 45.339) (end 328.3204 43.1546) (width 0.508) (layer B.Cu) (net 17))
   (segment (start 328.3204 43.1546) (end 328.3204 40.5638) (width 0.508) (layer B.Cu) (net 17))
   (segment (start 322.072 80.772) (end 326.136 76.708) (width 0.508) (layer B.Cu) (net 17))
-  (segment (start 326.136 76.708) (end 326.136 45.339) (width 0.508) (layer B.Cu) (net 17))
+  (segment (start 326.136 76.708) (end 326.136 46.482) (width 0.508) (layer B.Cu) (net 17))
+  (segment (start 326.136 46.482) (end 326.136 45.339) (width 0.508) (layer B.Cu) (net 17))
   (segment (start 320.802 82.042) (end 322.072 80.772) (width 0.508) (layer B.Cu) (net 17))
   (segment (start 320.294 82.55) (end 320.802 82.042) (width 0.508) (layer B.Cu) (net 17))

Commit message: Multiple pad revisions after inspecting prototype.
Extended pads for BD_D1, USB MINI-B.
Increased hole and pad size for BC_Ct1 and BC_D1.

The old sizes work fine but this will make it easier to solder, give
some extra wiggle room.
Routing:
- net N-00000112: track 15.7 -> 17.7 mm
- net /GND: track 204.2 -> 203.3 mm

Commit message: Fixed error with boost converter wiring for BC_R1 found in prototype.
On the prototype this is an easy fix, basically you can just rotate the
resistor to the side and solder it to the same pin the trace goes to in
the diagram now.
Connections:
- BC_R1 pad 1: /LEDCOL0 -> N-00000105
- BC_R2 pad 1: N-00000115 (its old number) -> N-00000105
- VREG1 pad 5: N-00000115 (its old number) -> N-00000105
Routing:
- net N-00000105: track 0.00 -> 53.9 mm, vias 0 -> 4
- net N-00000115 (its old number): track 44.7 -> 0.00 mm, vias 3 -> 0
- net /LEDCOL0: track 738.1 -> 731.6 mm
